File: end_plates/end_plate_ctrl.kicad_pcb (KiCad board)
At the start: 2 copper layers, 103 x 53 mm, 9 parts

Commit message: Added README.md and project_outputs
Changed lines of the file:
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@@
     (visible_elements FFFFFF7F)
     (pcbplotparams
-      (layerselection 0x00020_7ffffffe)
+      (layerselection 0x01030_ffffffff)
       (usegerberextensions false)
       (usegerberattributes false)
@@
       (padsonsilk false)
       (subtractmaskfromsilk false)
-      (outputformat 3)
+      (outputformat 1)
       (mirror false)
       (drillshape 0)
       (scaleselection 1)
-      (outputdirectory ""))
+      (outputdirectory "../project_outputs/end_plate_ctrl/"))
   )
   (net 0 "")
@@
     (uvia_dia 0.3)
     (uvia_drill 0.1)
+  )
+  (module footprints:DB9_end_plate (layer F.Cu)
+    (at 178.5 86.14)
+    (fp_text reference "Hand controller" (at 0 5) (layer F.SilkS)
+      (effects (font (size 3 2.8) (thickness 0.5)))
+    )
+    (fp_text value DB9_end_plate (at 0 -14) (layer F.Fab)
+      (effects (font (size 1 1) (thickness 0.15)))
+    )
+    (fp_line (start -8 -0.8) (end -8 -11.8) (layer F.Fab) (width 0.05))
+    (fp_line (start -8 -0.8) (end 8 -0.8) (layer F.Fab) (width 0.05))
+    (fp_line (start 8 -0.8) (end 8 -11.8) (layer F.Fab) (width 0.05))
+    (fp_line (start -8 -11.8) (end 8 -11.8) (layer F.Fab) (width 0.05))
+    (fp_line (start -17 -6.3) (end 17 -6.3) (layer F.Fab) (width 0.05))
+    (fp_line (start -17 -13) (end 17 -13) (layer B.CrtYd) (width 0.1))
+    (fp_line (start 17 -13) (end 17 9) (layer B.CrtYd) (width 0.1))
+    (fp_line (start 17 9) (end -17 9) (layer B.CrtYd) (width 0.1))
+    (fp_line (start -17 9) (end -17 -13) (layer B.CrtYd) (width 0.1))
+    (pad "" np_thru_hole oval (at 0 -6.3) (size 31.2 6.7) (drill oval 31.2 6.7) (layers *.Cu *.Mask))
+    (pad "" np_thru_hole oval (at 0 -2.8) (size 18 4) (drill oval 18 4) (layers *.Cu *.Mask))
+    (pad "" np_thru_hole oval (at 0 -9.8) (size 18 4) (drill oval 18 4) (layers *.Cu *.Mask))
   )
   (module footprints:USB_B_flange (layer F.Cu)
@@
     (pad "" np_thru_hole oval (at 0 -10.9) (size 12.3 0.5) (drill oval 12.3 0.5) (layers *.Cu *.Mask))
   )
-  (module footprints:DB9_end_plate (layer F.Cu)
-    (at 178.5 86.14)
-    (fp_text reference "Hand controller" (at 0 5) (layer F.SilkS)
-      (effects (font (size 3 2.8) (thickness 0.5)))
-    )
-    (fp_text value DB9_end_plate (at 0 -14) (layer F.Fab)
-      (effects (font (size 1 1) (thickness 0.15)))
-    )
-    (fp_line (start -17 9) (end -17 -13) (layer B.CrtYd) (width 0.1))
-    (fp_line (start 17 9) (end -17 9) (layer B.CrtYd) (width 0.1))
-    (fp_line (start 17 -13) (end 17 9) (layer B.CrtYd) (width 0.1))
-    (fp_line (start -17 -13) (end 17 -13) (layer B.CrtYd) (width 0.1))
-    (fp_line (start -17 -6.3) (end 17 -6.3) (layer F.Fab) (width 0.05))
-    (fp_line (start -8 -11.8) (end 8 -11.8) (layer F.Fab) (width 0.05))
-    (fp_line (start 8 -0.8) (end 8 -11.8) (layer F.Fab) (width 0.05))
-    (fp_line (start -8 -0.8) (end 8 -0.8) (layer F.Fab) (width 0.05))
-    (fp_line (start -8 -0.8) (end -8 -11.8) (layer F.Fab) (width 0.05))
-    (pad "" np_thru_hole oval (at 0 -2.8) (size 16 2) (drill oval 16 2) (layers *.Cu *.Mask))
-    (pad "" np_thru_hole oval (at 0 -9.8) (size 18 4) (drill oval 18 4) (layers *.Cu *.Mask))
-    (pad "" np_thru_hole oval (at 0 -2.8) (size 18 4) (drill oval 18 4) (layers *.Cu *.Mask))
-    (pad "" np_thru_hole oval (at 0 -6.3) (size 31.2 6.7) (drill oval 31.2 6.7) (layers *.Cu *.Mask))
-  )
   (module footprints:NC5MBH_flange (layer F.Cu)
