File: onstep_pcb/onstep.kicad_pcb (KiCad board)
At the start: 2 copper layers, 120 x 100 mm, 137 parts, among them X1 "USB", X2 Battery Holder, X3 "FUSE", X4 Conn_01x09

Commit message: Added README.md and project_outputs
Parts:
- D1, D6: value MCP1700T_SOT-23 -> MCP1700
- D12: value MCP1700T_SOT-23 -> MCP1700T
- D13, D3, D8: value TMC2130-TA -> TMC2130
- D7: value FT230XS -> FT230
Other:
- rule pad_to_mask_clearance: 0.05 -> 0.07
